Commit message: ran on gazebo and live time change in rviz

File: description/robot_core.xacro (robot description, xacro)
@@ -1,4 +1,4 @@
 <?xml version="1.0"?>
-<robot xmlns:xacro="http://www.ros.org/wiki/xacro" >
+<robot xmlns:xacro="http://www.ros.org/wiki/xacro">
     <xacro:include filename="inertial_macros.xacro"/>
     <material name="white">
@@ -38,7 +38,10 @@
         </collision>
         <xacro:inertial_box mass="0.5" x="0.3" y="0.3" z="0.15">
-            <orogin xyz="0.15 0 0.075" rpy="0 0 0"/>
+            <origin xyz="0.15 0 0.075" rpy="0 0 0"/>
         </xacro:inertial_box>
     </link>
+    <gazebo reference="chassis">
+        <material>Gazebo/White</material>
+    </gazebo>
     <!-- LEFT WHEEL LINK -->
     <joint name="left_wheel_joint" type="continuous">
@@ -64,4 +67,7 @@
         </xacro:inertial_cylinder>
     </link>
+    <gazebo reference="left_wheel">
+        <material>Gazebo/Blue</material>
+    </gazebo>
         <!-- RIGHT WHEEL LINK -->
         <joint name="right_wheel_joint" type="continuous">
@@ -87,4 +93,7 @@
             </xacro:inertial_cylinder>
         </link>
+        <gazebo reference="right_wheel">
+            <material>Gazebo/Blue</material>
+        </gazebo>
         <!--CASTER WHEEL LINK-->
         <joint name="caster_wheel_joint" type="fixed">
@@ -109,3 +118,8 @@
             </xacro:inertial_sphere>
         </link>
+        <gazebo reference="caster_wheel">
+            <material>Gazebo/Black</material>
+            <mu1 value="0.001"/>
+            <mu2 value="0.001"/>
+        </gazebo>
 </robot>
